Commit message: update

File: src/dummy_ros2/urdf/dummy_ros2.urdf (robot description, URDF)
Before this commit: robot dummy_ros2, 7 links, 6 joints
Joints:
- joint Joint1: limit lower=-3.14 upper=3.14 effort=0 velocity=0 -> lower=-3.14 upper=3.14 effort=100 velocity=1.0
- joint Joint2: limit lower=-3.14 upper=3.14 effort=0 velocity=0 -> lower=-3.14 upper=3.14 effort=100 velocity=1.0
- joint Joint3: limit lower=-3.14 upper=3.14 effort=0 velocity=0 -> lower=-3.14 upper=3.14 effort=100 velocity=1.0
- joint Joint4: limit lower=-3.14 upper=3.14 effort=0 velocity=0 -> lower=-3.14 upper=3.14 effort=100 velocity=1.0
- joint Joint5: limit lower=-3.14 upper=3.14 effort=0 velocity=0 -> lower=-3.14 upper=3.14 effort=100 velocity=1.0
- joint Joint6: limit lower=-3.14 upper=3.14 effort=0 velocity=0 -> lower=-3.14 upper=3.14 effort=100 velocity=1.0
